File: Morse_code_PCB/Morse_code_PCB.kicad_sch (KiCad schematic)
At the start: 1 part

Commit message: 画了一点PCB Signed-off-by: kevin <kevin@lmve.net>
Parts:
- added C1: 100nF, Capacitor_SMD:C_0805_2012Metric, symbol Device:C
- added C2, C3: 10nF, Capacitor_SMD:C_0603_1608Metric, symbol Device:C
- added L1: 100mH, Inductor_SMD:L_0805_2012Metric, symbol Device:L
- added R1: 1K, Resistor_SMD:R_0603_1608Metric, symbol Device:R
- added R2, R3, R4: 10K, Resistor_SMD:R_0603_1608Metric, symbol Device:R
- added SW1: RotaryEncoder_Switch, MY:EC11, symbol Device:RotaryEncoder_Switch
- gave numbers to parts that had none: 1
Connections:
- net at U1.1 (BOOT0): now also R1.2
- net at U1.12 (PA6): now also C2.1, R3.1, SW1.A
- net at U1.13 (PA7): now also C3.1, R4.1, SW1.B
- net SW1: now reaches U1.14 (PB1)
- net SW1: now also SW1.S1
- net GND: now reaches U1.15 (VSS)
- net GND: now also C1.2, C2.2, C3.2, R1.1, SW1.C, SW1.S2
- net VCC: now reaches U1.16 (VDD)
- net VCC: now also L1.1, R2.2, R3.2, R4.2
- net at U1.4 (NRST): now also C1.1, R2.1
- net at U1.5 (VDDA): now also L1.2

Commit message: updata PCB Signed-off-by: kevin <kevin@lmve.net>
Parts:
- added J1: USB_C_Receptacle_USB2.0, Connector_USB:USB_C_Receptacle_HRO_TYPE-C-31-M-12, symbol Connector:USB_C_Receptacle_USB2.0
- added J2, J3: AudioJack3_Ground, Connector_Audio:Jack_3.5mm_PJ320D_Horizontal, symbol Connector:AudioJack3_Ground
Connections:
- new net: J1.A1 (GND), J1.A12 (GND), J1.B1 (GND), J1.B12 (GND)
- new net: J1.A4 (VBUS), J1.A9 (VBUS), J1.B4 (VBUS), J1.B9 (VBUS)
Changed lines of the file:
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@@
     (pin "1")
+  )
+  (symbol (lib_id "Connector:USB_C_Receptacle_USB2.0") (at 34.29 45.72 0) (unit 1)
+    (in_bom yes) (on_board yes) (fields_autoplaced)
+    (property "Reference" "J1" (id 0) (at 34.29 22.86 0))
+    (property "Value" "USB_C_Receptacle_USB2.0" (id 1) (at 34.29 25.4 0))
+    (property "Footprint" "Connector_USB:USB_C_Receptacle_HRO_TYPE-C-31-M-12" (id 2) (at 38.1 45.72 0)
+      (effects (font (size 1.27 1.27)) hide)
+    )
+    (property "Datasheet" "https://www.usb.org/sites/default/files/documents/usb_type-c.zip" (id 3) (at 38.1 45.72 0)
+      (effects (font (size 1.27 1.27)) hide)
+    )
+    (pin "A1")
+    (pin "A12")
+    (pin "A4")
+    (pin "A5")
+    (pin "A6")
+    (pin "A7")
+    (pin "A8")
+    (pin "A9")
+    (pin "B1")
+    (pin "B12")
+    (pin "B4")
+    (pin "B5")
+    (pin "B6")
+    (pin "B7")
+    (pin "B8")
+    (pin "B9")
+    (pin "S1")
   )
   (symbol (lib_id "Device:R") (at 86.36 92.71 180) (unit 1)
@@
     (pin "1")
     (pin "2")
+  )
+  (symbol (lib_id "Connector:AudioJack3_Ground") (at 138.43 30.48 0) (unit 1)
+    (in_bom yes) (on_board yes) (fields_autoplaced)
+    (property "Reference" "J3" (id 0) (at 136.525 21.59 0))
+    (property "Value" "AudioJack3_Ground" (id 1) (at 136.525 24.13 0))
+    (property "Footprint" "Connector_Audio:Jack_3.5mm_PJ320D_Horizontal" (id 2) (at 138.43 30.48 0)
+      (effects (font (size 1.27 1.27)) hide)
+    )
+    (property "Datasheet" "~" (id 3) (at 138.43 30.48 0)
+      (effects (font (size 1.27 1.27)) hide)
+    )
+    (pin "G")
+    (pin "R")
+    (pin "S")
+    (pin "T")
+  )
+  (symbol (lib_id "Connector:AudioJack3_Ground") (at 115.57 30.48 0) (unit 1)
+    (in_bom yes) (on_board yes) (fields_autoplaced)
+    (property "Reference" "J2" (id 0) (at 113.665 21.59 0))
+    (property "Value" "AudioJack3_Ground" (id 1) (at 113.665 24.13 0))
+    (property "Footprint" "Connector_Audio:Jack_3.5mm_PJ320D_Horizontal" (id 2) (at 115.57 30.48 0)
+      (effects (font (size 1.27 1.27)) hide)
+    )
+    (property "Datasheet" "~" (id 3) (at 115.57 30.48 0)
+      (effects (font (size 1.27 1.27)) hide)
+    )
+    (pin "G")
+    (pin "R")
+    (pin "S")
+    (pin "T")
   )
   (symbol (lib_id "power:VCC") (at 81.28 67.31 0) (unit 1)
@@
       (reference "C3") (unit 1) (value "10nF") (footprint "Capacitor_SMD:C_0603_1608Metric")
     )
+    (path "/5c470add-b449-455e-95fc-baae46d35c85"
+      (reference "J1") (unit 1) (value "USB_C_Receptacle_USB2.0") (footprint "Connector_USB:USB_C_Receptacle_HRO_TYPE-C-31-M-12")
+    )
+    (path "/9b532d94-5adf-40a9-aa2f-bc58284f6753"
+      (reference "J2") (unit 1) (value "AudioJack3_Ground") (footprint "Connector_Audio:Jack_3.5mm_PJ320D_Horizontal")
+    )
+    (path "/93b86c17-095d-4de5-a8b5-bb4c5838f14a"
+      (reference "J3") (unit 1) (value "AudioJack3_Ground") (footprint "Connector_Audio:Jack_3.5mm_PJ320D_Horizontal")
+    )
     (path "/a6e73968-bfeb-49ba-b5d0-6a71117f7ee3"

Commit message: 画了个12864OLED封装 Signed-off-by: kevin <kevin@lmve.net>
Parts:
- added U2: OLED_12864, MY:OLED12864, symbol MY:OLED_12864
Changed lines of the file:
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@@
     )
+  )
+  (symbol (lib_id "MY:OLED_12864") (at 160.02 46.99 0) (unit 1)
+    (in_bom yes) (on_board yes) (fields_autoplaced)
+    (property "Reference" "U2" (id 0) (at 173.99 49.5299 0)
+      (effects (font (size 1.27 1.27)) (justify left))
+    )
+    (property "Value" "OLED_12864" (id 1) (at 173.99 52.0699 0)
+      (effects (font (size 1.27 1.27)) (justify left))
+    )
+    (property "Footprint" "MY:OLED12864" (id 2) (at 160.02 46.99 0)
+      (effects (font (size 1.27 1.27)) hide)
+    )
+    (property "Datasheet" "" (id 3) (at 160.02 46.99 0)
+      (effects (font (size 1.27 1.27)) hide)
+    )
+    (pin "1")
+    (pin "2")
+    (pin "3")
+    (pin "4")
   )
   (symbol (lib_id "Device:R") (at 137.16 87.63 180) (unit 1)
@@
       (reference "U1") (unit 1) (value "STM32F030F4Px") (footprint "Package_SO:TSSOP-20_4.4x6.5mm_P0.65mm")
     )
-  )
+    (path "/114181eb-7392-4a8c-8162-9def16899b0d"
+      (reference "U2") (unit 1) (value "OLED_12864") (footprint "MY:OLED12864")
+    )
+  )

Commit message: 摸鱼画了一点 Signed-off-by: kevin <kevin@lmve.net>
Parts:
- added BZ?: Buzzer, Buzzer_Beeper:Buzzer_TDK_PS1240P02BT_D12.2mm_H6.5mm, symbol Device:Buzzer
- added C? (x4): 10uF, Capacitor_SMD:C_2220_5650Metric, symbol Device:C
- added C? (x4): 104, Capacitor_SMD:C_0805_2012Metric, symbol Device:C
- added D? (x3): 1N4148WT, Diode_SMD:D_SOD-523, symbol Diode:1N4148WT
- added D? (x2): LED, LED_SMD:LED_0603_1608Metric, symbol Device:LED
- added Q? (x2): AO3401A, Package_TO_SOT_SMD:SOT-23, symbol Transistor_FET:AO3401A
- added Q? (x2): AO3400A, Package_TO_SOT_SMD:SOT-23, symbol Transistor_FET:AO3400A
- added R? (x2): 100, Resistor_SMD:R_0603_1608Metric, symbol Device:R
- added R? (x6): 10K, Resistor_SMD:R_0603_1608Metric, symbol Device:R
- added R? (x4): 20K, Resistor_SMD:R_0603_1608Metric, symbol Device:R
- added R?: 510, Resistor_SMD:R_0603_1608Metric, symbol Device:R
- added R? (x2): 2K, Resistor_SMD:R_0603_1608Metric, symbol Device:R
- added R?: 1K, Resistor_SMD:R_0603_1608Metric, symbol Device:R
- added R?: *R0, Resistor_SMD:R_0402_1005Metric, symbol Device:R
- added U?: MCP73831-2-OT, Package_TO_SOT_SMD:SOT-23-5, symbol Battery_Management:MCP73831-2-OT
- added U?: 24AA02-OT, Package_SO:TSSOP-8_4.4x3mm_P0.65mm, symbol Memory_EEPROM:24AA02-OT
- added U?: CH340E, Package_SO:MSOP-10_3x3mm_P0.5mm, symbol Interface_USB:CH340E
- added U?: LP5907MFX-3.3, Package_TO_SOT_SMD:SOT-23-5, symbol Regulator_Linear:LP5907MFX-3.3
Connections:
- net GND: now also J1.A1 (GND), J1.A12 (GND), J1.B1 (GND), J1.B12 (GND), U2.1 (GND), C?.2, C?.2, C?.2, C?.2, C?.2, C?.2, C?.2, C?.2, D?.1 (K), Q?.2 (S), Q?.2 (S), R?.1, R?.1, R?.2, R?.2, U?.2 (GND), U?.2 (GND), U?.2 (VSS), U?.3 (GND)
- net VCC: now also U2.2 (VCC), C?.1, C?.1, Q?.2 (S), R?.1, R?.1, R?.2, R?.2, R?.2, U?.4 (VCC), U?.5 (OUT), U?.7 (VCC)
- net IIC_SCL: now reaches U2.3 (SCL)
- net IIC_SCL: now also U1.17 (PA9), R?.1, U?.1 (SCL)
- net IIC_SDL: now reaches U2.4 (SDL)
- net IIC_SDL: now also U1.18 (PA10), R?.1, U?.3 (SDA)
- net at R1.2, U1.1 (BOOT0): now also R?.2
- net USB_VCC: now reaches J1.A4 (VBUS), J1.A9 (VBUS), J1.B4 (VBUS), J1.B9 (VBUS)
- net USB_VCC: now also C?.1, D?.2 (A), U?.4 (VDD)
- net at J1.A6 (D+): now also J1.B6 (D+), R?.2
- net at J1.A7 (D-): now also J1.B7 (D-), R?.2
- new net: R?.1, R?.2, U?.1 (UD+)
- new net: Q?.1 (G), R?.1, R?.2 (x2)
- new net: D?.2 (A), Q?.1 (G), Q?.3 (D), R?.1
- new net: D?.1 (K), Q?.1 (G), R?.1
- new net: R?.1, U?.2 (UD-)
- new net: R?.1, U?.6 (TNOW)
- new net: D?.2 (A), R?.2
- new net: C?.1, U?.10 (V3)
- new net: BZ?.1 (-), Q?.3 (D)
- new net: BZ?.2 (+), Q?.3 (D)
- new net: D?.1 (K), R?.1
- new net: R?.2, U?.5 (PROG)
- new net BAT: C?.1, C?.1, Q?.3 (D), R?.1, U?.1 (IN), U?.3 (EN)
- new net BAT_ADC: R?.1, R?.2
- new net BAT_CHG_DET: R?.2, U?.1 (STAT)
- new net BAT_IN: C?.1, C?.1, Q?.2 (S), R?.2, U?.3 (VBAT)
- new net K1: D?.1 (K), D?.1 (K)
- new net K1_DET: D?.2 (A)
- new net MUTE: R?.1
- new net PWM: R?.2
- new net PWR_EN: D?.2 (A)
Other:
- moved on the sheet: C1, C2, C3, J1, J2, J3, L1, R1, R2, R3, R4, SW1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

Commit message: updata Signed-off-by: kevin <kevin@lmve.net>
Parts:
- C10, C5, C6, C8: renamed from C?; footprint Capacitor_SMD:C_2220_5650Metric -> Capacitor_SMD:C_1206_3216Metric
- gave numbers to parts that had none: 35
Connections:
- net GND: now also J2.R2, J3.R2
- net TXD: now reaches U4.8 (TXD)
- net RXD: now reaches U4.9 (RXD)

Commit message: updata PCB
Parts:
- added C? (x2): 10uF, Capacitor_SMD:C_1206_3216Metric, symbol Device:C
- added D?: LED, LED_SMD:LED_0603_1608Metric, symbol Device:LED
- added R? (x3): 20K, Resistor_SMD:R_0603_1608Metric, symbol Device:R
- J2: value AudioJack3_Ground -> INPUT
- J3: value AudioJack3_Ground -> OUTPUT
Connections:
- net GND: now also D?.1 (K)
- net K1: now also SW1.S1
- net K1_DET: now also U1.14 (PB1)
- net PWM: now also C?.2, C?.2
- net VCC: now also R?.1, R?.1
- net at J3.R1: now also C?.1
- net at J3.T: now also C?.1
- net TICK_A: now reaches J2.R1
- net TICK_A: now also R?.2
- net TICK_B: now reaches J2.T
- net TICK_B: now also R?.2
- removed net SW1: SW1.S1, U1.14 (PB1)
- new net: D?.2 (A), R?.2
- new net RUN_LED: R?.1
Other:
- moved on the sheet: J3

Commit message: UPDATA PCB Signed-off-by: kevin <kevin@lmve.net>
Parts:
- R22, R23: renamed from R?; value 20K -> 1K
- R24: renamed from R?; value 20K -> 510
- gave numbers to parts that had none: 3
Connections:
- net BAT_ADC: now also U1.6 (PA0)
- net BAT_CHG_DET: now also U1.7 (PA1)
- net MUTE: now also U1.11 (PA5)
- net PWM: now also U1.10 (PA4)
- net PWR_EN: now also U1.19 (PA13)
- net RUN_LED: now also U1.20 (PA14)
- net RXD: now also U1.8 (PA2)
- net TICK_A: now also U1.2 (PF0)
- net TICK_B: now also U1.3 (PF1)
- net TXD: now also U1.9 (PA3)
- net BAT: no longer names the net of C8.1, C9.1, Q2.3 (D), R8.1, U5.1 (IN), U5.3 (EN)
Other:
- moved on the sheet: D6, R24

Commit message: UPDATA PCB Signed-off-by: kevin <kevin@lmve.net>
Parts:
- added J4: Conn_01x02_Female, MY:SIP-2, symbol Connector:Conn_01x02_Female
- U6: footprint Package_SO:TSSOP-8_4.4x3mm_P0.65mm -> Package_TO_SOT_SMD:SOT-23-5
Connections:
- net BAT_IN: now also J4.1 (Pin_1)
- net GND: now also J1.S1 (SHIELD), J4.2 (Pin_2)
Changed lines of the file:
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@@
+    )
+  )
+  (global_label "BAT_IN" (shape input) (at 145.415 135.255 180) (fields_autoplaced)
+    (effects (font (size 1.27 1.27)) (justify right))
+    (property "Intersheet References" "${INTERSHEET_REFS}" (id 0) (at 136.7729 135.1756 0)
+      (effects (font (size 1.27 1.27)) (justify right) hide)
     )
   )
@@
     (pin "3")
     (pin "4")
+  )
+  (symbol (lib_id "Connector:Conn_01x02_Female") (at 150.495 135.255 0) (unit 1)
+    (in_bom yes) (on_board yes) (fields_autoplaced)
+    (property "Reference" "J4" (id 0) (at 152.4 135.2549 0)
+      (effects (font (size 1.27 1.27)) (justify left))
+    )
+    (property "Value" "Conn_01x02_Female" (id 1) (at 152.4 137.7949 0)
+      (effects (font (size 1.27 1.27)) (justify left))
+    )
+    (property "Footprint" "MY:SIP-2" (id 2) (at 150.495 135.255 0)
+      (effects (font (size 1.27 1.27)) hide)
+    )
+    (property "Datasheet" "~" (id 3) (at 150.495 135.255 0)
+      (effects (font (size 1.27 1.27)) hide)
+    )
+    (pin "1")
+    (pin "2")
   )
   (symbol (lib_id "Device:R") (at 166.37 40.64 180) (unit 1)
@@
     (pin "S1")
     (pin "S2")
+  )
+  (symbol (lib_id "power:GND") (at 17.78 59.055 0) (unit 1)
+    (in_bom yes) (on_board yes)
+    (property "Reference" "#PWR0119" (id 0) (at 17.78 65.405 0)
+      (effects (font (size 1.27 1.27)) hide)
+    )
+    (property "Value" "GND" (id 1) (at 17.78 62.865 0))
+    (property "Footprint" "" (id 2) (at 17.78 59.055 0)
+      (effects (font (size 1.27 1.27)) hide)
+    )
+    (property "Datasheet" "" (id 3) (at 17.78 59.055 0)
+      (effects (font (size 1.27 1.27)) hide)
+    )
+    (pin "1")
   )
   (symbol (lib_id "Device:C") (at 162.56 66.04 0) (unit 1)
@@
     (pin "2")
   )
+  (symbol (lib_id "Memory_EEPROM:24AA02-OT") (at 219.71 53.34 0) (unit 1)
+    (in_bom yes) (on_board yes) (fields_autoplaced)
+    (property "Reference" "U6" (id 0) (at 210.82 52.0699 0)
+      (effects (font (size 1.27 1.27)) (justify right))
+    )
+    (property "Value" "24AA02-OT" (id 1) (at 210.82 54.6099 0)
+      (effects (font (size 1.27 1.27)) (justify right))
+    )
+    (property "Footprint" "Package_TO_SOT_SMD:SOT-23-5" (id 2) (at 219.71 53.34 0)
+      (effects (font (size 1.27 1.27)) hide)
+    )
+    (property "Datasheet" "http://ww1.microchip.com/downloads/en/DeviceDoc/21709J.pdf" (id 3) (at 219.71 53.34 0)
+      (effects (font (size 1.27 1.27)) hide)
+    )
+    (pin "1")
+    (pin "2")
+    (pin "3")
+    (pin "4")
+    (pin "5")
+  )
   (symbol (lib_id "Device:R") (at 44.45 114.935 0) (unit 1)
     (in_bom yes) (on_board yes)
@@
     (pin "2")
   )
+  (symbol (lib_id "power:GND") (at 145.415 137.795 0) (unit 1)
+    (in_bom yes) (on_board yes) (fields_autoplaced)
+    (property "Reference" "#PWR03" (id 0) (at 145.415 144.145 0)
+      (effects (font (size 1.27 1.27)) hide)
+    )
+    (property "Value" "GND" (id 1) (at 145.415 142.875 0))
+    (property "Footprint" "" (id 2) (at 145.415 137.795 0)
+      (effects (font (size 1.27 1.27)) hide)
+    )
+    (property "Datasheet" "" (id 3) (at 145.415 137.795 0)
+      (effects (font (size 1.27 1.27)) hide)
+    )
+    (pin "1")
+  )
   (symbol (lib_id "power:VCC") (at 99.06 20.32 0) (unit 1)
     (in_bom yes) (on_board yes) (fields_autoplaced)
@@
     (pin "1")
     (pin "2")
-  )
-  (symbol (lib_id "Memory_EEPROM:24AA02-OT") (at 219.71 53.34 0) (unit 1)
-    (in_bom yes) (on_board yes) (fields_autoplaced)
-    (property "Reference" "U6" (id 0) (at 210.82 52.0699 0)
-      (effects (font (size 1.27 1.27)) (justify right))
-    )
-    (property "Value" "24AA02-OT" (id 1) (at 210.82 54.6099 0)
-      (effects (font (size 1.27 1.27)) (justify right))
-    )
-    (property "Footprint" "Package_SO:TSSOP-8_4.4x3mm_P0.65mm" (id 2) (at 219.71 53.34 0)
-      (effects (font (size 1.27 1.27)) hide)
-    )
-    (property "Datasheet" "http://ww1.microchip.com/downloads/en/DeviceDoc/21709J.pdf" (id 3) (at 219.71 53.34 0)
-      (effects (font (size 1.27 1.27)) hide)
-    )
-    (pin "1")
-    (pin "2")
-    (pin "3")
-    (pin "4")
-    (pin "5")
   )
   (symbol (lib_id "Device:R") (at 104.14 30.48 0) (unit 1)
@@
       (reference "#PWR02") (unit 1) (value "GND") (footprint "")
     )
+    (path "/a4d12d50-8ee9-42d1-ba1f-da61fb555338"
+      (reference "#PWR03") (unit 1) (value "GND") (footprint "")
+    )
     (path "/4d3fbe30-8d80-40e0-b7ae-5eda5664f629"
       (reference "#PWR0101") (unit 1) (value "GND") (footprint "")
@@
       (reference "#PWR0118") (unit 1) (value "GND") (footprint "")
     )
+    (path "/15ae5f90-ccc7-4e15-adc6-ac3e5518b056"
+      (reference "#PWR0119") (unit 1) (value "GND") (footprint "")
+    )
     (path "/972eb069-8d6d-41f6-83d3-1d7e45627208"
       (reference "BZ1") (unit 1) (value "Buzzer") (footprint "Buzzer_Beeper:Buzzer_TDK_PS1240P02BT_D12.2mm_H6.5mm")
@@
       (reference "J3") (unit 1) (value "OUTPUT") (footprint "Connector_Audio:Jack_3.5mm_PJ320D_Horizontal")
     )
+    (path "/13d1db83-c817-49c7-a180-de3dec8b3297"
+      (reference "J4") (unit 1) (value "Conn_01x02_Female") (footprint "MY:SIP-2")
+    )
     (path "/a6e73968-bfeb-49ba-b5d0-6a71117f7ee3"
       (reference "L1") (unit 1) (value "100mH") (footprint "Inductor_SMD:L_0805_2012Metric")
@@
       (reference "U5") (unit 1) (value "LP5907MFX-3.3") (footprint "Package_TO_SOT_SMD:SOT-23-5")
     )
-    (path "/be287c62-1fc6-4a9d-b9ca-596c13d522fb"
-      (reference "U6") (unit 1) (value "24AA02-OT") (footprint "Package_SO:TSSOP-8_4.4x3mm_P0.65mm")
-    )
-  )
+    (path "/86071cfe-1543-479d-bd7a-9553562bc5e9"
+      (reference "U6") (unit 1) (value "24AA02-OT") (footprint "Package_TO_SOT_SMD:SOT-23-5")
+    )
+  )
