File: Morse_code_PCB/Morse_code_PCB.kicad_sch (KiCad schematic)
At the start: 60 parts, among them J1 USB_C_Receptacle_USB2.0, J2 INPUT, J3 OUTPUT, J4 Conn_01x02_Female, Q1 AO3400A, Q2 AO3401A, Q3 AO3400A, Q4 AO3401A, SW1 RotaryEncoder_Switch, U1 STM32F030F4Px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

Commit message: PCB画完 Signed-off-by: kevin <kevin@lmve.net>
Parts:
- added J5: Conn_01x04_Female, MY:SIP-4, symbol Connector:Conn_01x04_Female
Connections:
- net GND: now also J5.2 (Pin_2)
- net PWR_EN: now also J5.3 (Pin_3)
- net RUN_LED: now also J5.4 (Pin_4)
- net VCC: now also J5.1 (Pin_1)
Changed lines of the file:
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@@
+    )
+  )
+  (global_label "RUN_LED" (shape input) (at 142.875 115.57 180) (fields_autoplaced)
+    (effects (font (size 1.27 1.27)) (justify right))
+    (property "插入图纸页参考" "${INTERSHEET_REFS}" (id 0) (at 132.1162 115.6494 0)
+      (effects (font (size 1.27 1.27)) (justify right) hide)
     )
   )
@@
     (property "插入图纸页参考" "${INTERSHEET_REFS}" (id 0) (at 64.6431 181.5306 0)
       (effects (font (size 1.27 1.27)) (justify left) hide)
+    )
+  )
+  (global_label "PWR_EN" (shape input) (at 142.875 113.03 180) (fields_autoplaced)
+    (effects (font (size 1.27 1.27)) (justify right))
+    (property "Intersheet References" "${INTERSHEET_REFS}" (id 0) (at 133.0233 113.1094 0)
+      (effects (font (size 1.27 1.27)) (justify right) hide)
     )
   )
@@
     (pin "8")
     (pin "9")
+  )
+  (symbol (lib_id "power:VCC") (at 142.875 107.95 90) (unit 1)
+    (in_bom yes) (on_board yes)
+    (property "Reference" "#PWR0121" (id 0) (at 146.685 107.95 0)
+      (effects (font (size 1.27 1.27)) hide)
+    )
+    (property "Value" "VCC" (id 1) (at 139.065 107.95 0))
+    (property "Footprint" "" (id 2) (at 142.875 107.95 0)
+      (effects (font (size 1.27 1.27)) hide)
+    )
+    (property "Datasheet" "" (id 3) (at 142.875 107.95 0)
+      (effects (font (size 1.27 1.27)) hide)
+    )
+    (pin "1")
   )
   (symbol (lib_id "Device:R") (at 48.895 36.83 270) (unit 1)
@@
     (pin "2")
   )
+  (symbol (lib_id "power:GND") (at 142.875 110.49 270) (unit 1)
+    (in_bom yes) (on_board yes)
+    (property "Reference" "#PWR0120" (id 0) (at 136.525 110.49 0)
+      (effects (font (size 1.27 1.27)) hide)
+    )
+    (property "Value" "GND" (id 1) (at 139.065 110.49 0))
+    (property "Footprint" "" (id 2) (at 142.875 110.49 0)
+      (effects (font (size 1.27 1.27)) hide)
+    )
+    (property "Datasheet" "" (id 3) (at 142.875 110.49 0)
+      (effects (font (size 1.27 1.27)) hide)
+    )
+    (pin "1")
+  )
   (symbol (lib_id "Transistor_FET:AO3401A") (at 246.38 71.755 180) (unit 1)
     (in_bom yes) (on_board yes)
@@
     (pin "1")
     (pin "2")
+  )
+  (symbol (lib_id "Connector:Conn_01x04_Female") (at 147.955 110.49 0) (unit 1)
+    (in_bom yes) (on_board yes) (fields_autoplaced)
+    (property "Reference" "J5" (id 0) (at 149.86 110.4899 0)
+      (effects (font (size 1.27 1.27)) (justify left))
+    )
+    (property "Value" "Conn_01x04_Female" (id 1) (at 149.86 113.0299 0)
+      (effects (font (size 1.27 1.27)) (justify left))
+    )
+    (property "Footprint" "MY:SIP-4" (id 2) (at 147.955 110.49 0)
+      (effects (font (size 1.27 1.27)) hide)
+    )
+    (property "Datasheet" "~" (id 3) (at 147.955 110.49 0)
+      (effects (font (size 1.27 1.27)) hide)
+    )
+    (pin "1")
+    (pin "2")
+    (pin "3")
+    (pin "4")
   )
   (symbol (lib_id "Device:R") (at 234.95 100.33 180) (unit 1)
@@
       (reference "#PWR0119") (unit 1) (value "GND") (footprint "")
     )
+    (path "/8db05113-bb5d-40cb-916f-5b0147562482"
+      (reference "#PWR0120") (unit 1) (value "GND") (footprint "")
+    )
+    (path "/4bc53345-25fe-427a-a648-514d97b80f54"
+      (reference "#PWR0121") (unit 1) (value "VCC") (footprint "")
+    )
     (path "/972eb069-8d6d-41f6-83d3-1d7e45627208"
       (reference "BZ1") (unit 1) (value "Buzzer") (footprint "Buzzer_Beeper:Buzzer_TDK_PS1240P02BT_D12.2mm_H6.5mm")
@@
       (reference "J4") (unit 1) (value "Conn_01x02_Female") (footprint "MY:SIP-2")
     )
+    (path "/9f9d9ec1-f12a-47cb-a033-e6a9e0eb276a"
+      (reference "J5") (unit 1) (value "Conn_01x04_Female") (footprint "MY:SIP-4")
+    )
     (path "/a6e73968-bfeb-49ba-b5d0-6a71117f7ee3"

Commit message: PCB updata Signed-off-by: kevin <kevin@lmve.net>
Parts:
- added BT1: Battery_Cell, MY:BAT_BC501SM, symbol Device:Battery_Cell
- added U7: STM32F103C8Tx, Package_QFP:LQFP-48_7x7mm_P0.5mm, symbol MCU_ST_STM32F1:STM32F103C8Tx
- added Y1: 8M, Crystal:Crystal_SMD_5032-2Pin_5.0x3.2mm, symbol Device:Crystal
- added Y2: 32.768k, Crystal:Crystal_SMD_3215-2Pin_3.2x1.5mm, symbol Device:Crystal
Other:
- moved on the sheet: BZ1, C1, C2, C3, D6, J4, J5, L1, Q3, Q4, R1, R15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

Commit message: updata pcb
Parts:
- added C? (x3): C, Capacitor_SMD:C_0402_1005Metric_Pad0.74x0.62mm_HandSolder, symbol Device:C
- added C?: 100nF, Capacitor_SMD:C_0805_2012Metric, symbol Device:C
- added C?: (no value), symbol Device:C
- added L?: 100mH, Inductor_SMD:L_0805_2012Metric, symbol Device:L
- added R?: 1K, Resistor_SMD:R_0603_1608Metric, symbol Device:R
- added R?: 10K, Resistor_SMD:R_0603_1608Metric, symbol Device:R
- added R?: *R0, Resistor_SMD:R_0402_1005Metric, symbol Device:R
Connections:
- net BAT_ADC: now also U7.10 (PA0)
- net BAT_CHG_DET: now also U7.11 (PA1)
- net GND: now also BT1.2 (-), U7.23 (VSS), U7.35 (VSS), U7.47 (VSS), U7.8 (VSSA), C?.1, C?.1, C?.1, C?.1, C?.2, R?.1
- net IIC_SCL: now also U7.42 (PB6)
- net IIC_SDL: now also U7.43 (PB7)
- net PWR_EN: no longer J5.3 (Pin_3)
- net RUN_LED: no longer J5.4 (Pin_4)
- net RXD: now also U7.30 (PA9)
- net TXD: now also U7.31 (PA10)
- net VCC: now also U7.24 (VDD), U7.36 (VDD), U7.48 (VDD), L?.1, R?.1, R?.2
- net at U7.1 (VBAT): now also BT1.1 (+)
- net at U7.3 (PC14): now also Y2.2, C?.2
- net SW_D: now reaches U7.34 (PA13)
- net SW_D: now also J5.3 (Pin_3)
- net SW_L: now reaches U7.37 (PA14)
- net SW_L: now also J5.4 (Pin_4)
- net at U7.4 (PC15): now also Y2.1, C?.2
- net at U7.44 (BOOT0): now also R?.2, R?.2
- net at U7.5 (PD0): now also Y1.2, C?.2
- net at U7.6 (PD1): now also Y1.1, C?.2
- net at U7.7 (NRST): now also C?.1, R?.1
- net at U7.9 (VDDA): now also L?.2
Other:
- moved on the sheet: BT1, J5, U7, Y1, Y2

Commit message: Updata PCB Signed-off-by: kevin <kevin@lmve.net>
Parts:
- removed C1: 100nF, Capacitor_SMD:C_0805_2012Metric, symbol Device:C
- removed C4: 104, Capacitor_SMD:C_0805_2012Metric, symbol Device:C
- removed D2: LED, LED_SMD:LED_0603_1608Metric, symbol Device:LED
- removed L1: 100mH, Inductor_SMD:L_0805_2012Metric, symbol Device:L
- removed R1: 1K, Resistor_SMD:R_0603_1608Metric, symbol Device:R
- removed R14: 510, Resistor_SMD:R_0603_1608Metric, symbol Device:R
- removed R15: *R0, Resistor_SMD:R_0402_1005Metric, symbol Device:R
- removed R2: 10K, Resistor_SMD:R_0603_1608Metric, symbol Device:R
- removed U1: STM32F030F4Px, Package_SO:TSSOP-20_4.4x6.5mm_P0.65mm, symbol MCU_ST_STM32F0:STM32F030F4Px
- removed U4: CH340E, Package_SO:MSOP-10_3x3mm_P0.5mm, symbol Interface_USB:CH340E
- C15: renamed from C?; value (none) -> C; footprint (none) -> Capacitor_SMD:C_0402_1005Metric_Pad0.74x0.62mm_HandSolder
- gave numbers to parts that had none: 8
Connections:
- net K1_DET: now also U7.39 (PB3)
- net MUTE: now also U7.13 (PA3)
- net PWM: now also U7.12 (PA2)
- net PWR_EN: now also U7.29 (PA8)
- net RUN_LED: now also U7.28 (PB15)
- net TICK_A: now also U7.18 (PB0)
- net TICK_B: now also U7.19 (PB1)
- net VCC: now also R13.2; no longer R13.1
- net USB_DN: now reaches U7.32 (PA11)
- net USB_DN: now also R11.1
- net USB_DP: now reaches U7.33 (PA12)
- net USB_DP: now also R12.1
- net EN_A: now reaches U7.40 (PB4)
- net EN_A: now also C2.1, R3.1, SW1.A
- net EN_B: now reaches U7.41 (PB5)
- net EN_B: now also C3.1, R4.1, SW1.B
- net at J1.A6 (D+), J1.B6 (D+): now also R12.2, R13.1; no longer R11.2
- net at J1.A7 (D-), J1.B7 (D-): now also R11.2; no longer R12.2
Other:
- moved on the sheet: J1, R11, R12, R13
