File: Morse_code_PCB/Morse_code_PCB.kicad_pcb (KiCad board)
At the start: 2 copper layers, 6 parts, among them SW1 RotaryEncoder_Switch, U1 STM32F030F4Px

Commit message: updata PCB Signed-off-by: kevin <kevin@lmve.net>
Parts:
- added C2: 10nF, Capacitor_SMD:C_0603_1608Metric, F.Cu at (43.2, 165.1)
- added C3: 10nF, Capacitor_SMD:C_0603_1608Metric, F.Cu at (47.2, 165.1)
- added R3: 10K, Resistor_SMD:R_0603_1608Metric, F.Cu at (47.2, 162.6)
- added R4: 10K, Resistor_SMD:R_0603_1608Metric, F.Cu at (43.2, 162.6)
Connections:
- SW1 pad A: unconnected-(SW1-PadA) -> Net-(C2-Pad1)
- SW1 pad B: unconnected-(SW1-PadB) -> Net-(C3-Pad1)
- SW1 pad C: unconnected-(SW1-PadC) -> GND
- SW1 pad S1: unconnected-(SW1-PadS1) -> SW1
- SW1 pad S2: unconnected-(SW1-PadS2) -> GND
- U1 pad 12: unconnected-(U1-Pad12) -> Net-(C2-Pad1)
- U1 pad 13: unconnected-(U1-Pad13) -> Net-(C3-Pad1)
- U1 pad 14: unconnected-(U1-Pad14) -> SW1

Commit message: 屏蔽一些内容 Signed-off-by: kevin <kevin@lmve.net>
Parts:
- added J1: USB_C_Receptacle_USB2.0, Connector_USB:USB_C_Receptacle_HRO_TYPE-C-31-M-12, F.Cu at (56.9, 131.2)
- added J2: AudioJack3_Ground, Connector_Audio:Jack_3.5mm_PJ320D_Horizontal, F.Cu at (44.4, 142.0)
- added J3: AudioJack3_Ground, Connector_Audio:Jack_3.5mm_PJ320D_Horizontal, F.Cu at (44.4, 130.9)

Commit message: Signed-off-by: kevin <kevin@lmve.net>
Parts:
- moved J2 4.67 mm to (45.9, 137.5)
- moved J1 4.67 mm to (58.3, 126.8)
- moved J3 4.67 mm to (45.9, 126.5)
Changed lines of the file:
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@@
   (net 35 "unconnected-(J3-PadT)")
   (footprint "Connector_Audio:Jack_3.5mm_PJ320D_Horizontal" (layer "F.Cu")
-    (at 44.41 130.91)
+    (at 45.89 126.48)
     (descr "Headphones with microphone connector, 3.5mm, 4 pins (http://www.qingpu-electronics.com/en/products/WQP-PJ320D-72.html)")
     (tags "3.5mm jack mic microphone phones headphones 4pins audio plug")
@@
   )
   (footprint "Connector_Audio:Jack_3.5mm_PJ320D_Horizontal" (layer "F.Cu")
-    (at 44.41 141.96)
+    (at 45.89 137.53)
     (descr "Headphones with microphone connector, 3.5mm, 4 pins (http://www.qingpu-electronics.com/en/products/WQP-PJ320D-72.html)")
     (tags "3.5mm jack mic microphone phones headphones 4pins audio plug")
@@
   )
   (footprint "Connector_USB:USB_C_Receptacle_HRO_TYPE-C-31-M-12" (layer "F.Cu")
-    (at 56.85 131.18)
+    (at 58.33 126.75)
     (descr "USB Type-C receptacle for USB 2.0 and PD, http://www.krhro.com/uploads/soft/180320/1-1P320120243.pdf")
     (tags "usb usb-c 2.0 pd")

Commit message: 画了个12864OLED封装 Signed-off-by: kevin <kevin@lmve.net>
Parts:
- added U2: OLED_12864, MY:OLED12864, F.Cu at (78.8, 137.0)
Changed lines of the file:
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@@
   (net 34 "unconnected-(J3-PadS)")
   (net 35 "unconnected-(J3-PadT)")
+  (net 36 "unconnected-(U2-Pad1)")
+  (net 37 "unconnected-(U2-Pad2)")
+  (net 38 "unconnected-(U2-Pad3)")
+  (net 39 "unconnected-(U2-Pad4)")
   (footprint "Connector_Audio:Jack_3.5mm_PJ320D_Horizontal" (layer "F.Cu")
     (at 45.89 126.48)
@@
     )
   )
+  (footprint "MY:OLED12864" (layer "F.Cu")
+    (at 78.78 137.01)
+    (property "Sheetfile" "Morse_code_PCB.kicad_sch")
+    (property "Sheetname" "")
+    (attr through_hole)
+    (fp_text reference "U2" (at -5.5 -6.3 unlocked) (layer "F.SilkS")
+      (effects (font (size 1 1) (thickness 0.15)))
+    )
+    (fp_text value "OLED_12864" (at -5.5 -4.8 unlocked) (layer "F.Fab")
+      (effects (font (size 1 1) (thickness 0.15)))
+    )
+    (fp_text user "${REFERENCE}" (at -5.5 -3.3 unlocked) (layer "F.Fab")
+      (effects (font (size 1 1) (thickness 0.15)))
+    )
+    (fp_line (start 2 20) (end 2 3) (layer "F.SilkS") (width 0.12))
+    (fp_line (start 26 3) (end 26 20) (layer "F.SilkS") (width 0.12))
+    (fp_line (start 28 0) (end 0 0) (layer "F.SilkS") (width 0.12))
+    (fp_line (start 28 28) (end 28 0) (layer "F.SilkS") (width 0.12))
+    (fp_line (start 3 20) (end 2 20) (layer "F.SilkS") (width 0.12))
+    (fp_line (start 2 3) (end 26 3) (layer "F.SilkS") (width 0.12))
+    (fp_line (start 26 20) (end 3 20) (layer "F.SilkS") (width 0.12))
+    (fp_line (start 0 0) (end 0 28) (layer "F.SilkS") (width 0.12))
+    (fp_line (start 0 28) (end 28 28) (layer "F.SilkS") (width 0.12))
+    (pad "1" thru_hole rect (at 10.2 0.9) (size 1.524 1.524) (drill 1) (layers *.Cu *.Mask)
+      (net 36 "unconnected-(U2-Pad1)") (pinfunction "GND") (pintype "power_in"))
+    (pad "2" thru_hole circle (at 12.74 0.9) (size 1.524 1.524) (drill 1) (layers *.Cu *.Mask)
+      (net 37 "unconnected-(U2-Pad2)") (pinfunction "VCC") (pintype "power_in"))
+    (pad "3" thru_hole circle (at 15.28 0.9) (size 1.524 1.524) (drill 1) (layers *.Cu *.Mask)
+      (net 38 "unconnected-(U2-Pad3)") (pinfunction "SCL") (pintype "input"))
+    (pad "4" thru_hole circle (at 17.82 0.9) (size 1.524 1.524) (drill 1) (layers *.Cu *.Mask)
+      (net 39 "unconnected-(U2-Pad4)") (pinfunction "SDL") (pintype "input"))
+  )
   (footprint "MY:EC11" (layer "F.Cu")

Commit message: updata Signed-off-by: kevin <kevin@lmve.net>
Parts:
- added BZ1: Buzzer, Buzzer_Beeper:Buzzer_TDK_PS1240P02BT_D12.2mm_H6.5mm, F.Cu at (67.0, 142.7)
- added C10: 10uF, Capacitor_SMD:C_1206_3216Metric, F.Cu at (95.0, 120.5)
- added C11: 104, Capacitor_SMD:C_0805_2012Metric, F.Cu at (71.6, 151.1)
- added C4: 104, Capacitor_SMD:C_0805_2012Metric, F.Cu at (83.5, 143.6)
- added C5: 10uF, Capacitor_SMD:C_1206_3216Metric, F.Cu at (95.9, 127.5)
- added C6: 10uF, Capacitor_SMD:C_1206_3216Metric, F.Cu at (80.6, 138.6)
- added C7: 104, Capacitor_SMD:C_0805_2012Metric, F.Cu at (78.6, 148.0)
- added C8: 10uF, Capacitor_SMD:C_1206_3216Metric, F.Cu at (106.7, 118.1)
- added C9: 104, Capacitor_SMD:C_0805_2012Metric, F.Cu at (67.2, 151.1)
- added D1: 1N4148WT, Diode_SMD:D_SOD-523, F.Cu at (84.1, 151.7)
- added D2: LED, LED_SMD:LED_0603_1608Metric, F.Cu at (120.6, 107.8)
- added D3: LED, LED_SMD:LED_0603_1608Metric, F.Cu at (91.7, 136.7)
- added D4: 1N4148WT, Diode_SMD:D_SOD-523, F.Cu at (84.1, 149.2)
- added D5: 1N4148WT, Diode_SMD:D_SOD-523, F.Cu at (102.6, 132.2)
- added Q1: AO3400A, Package_TO_SOT_SMD:SOT-23, F.Cu at (102.5, 123.8)
- added Q2: AO3401A, Package_TO_SOT_SMD:SOT-23, F.Cu at (78.8, 144.3)
- added Q3: AO3400A, Package_TO_SOT_SMD:SOT-23, F.Cu at (87.2, 137.3)
- added Q4: AO3401A, Package_TO_SOT_SMD:SOT-23, F.Cu at (113.7, 113.5)
- added R10: 2K, Resistor_SMD:R_0603_1608Metric, F.Cu at (124.6, 110.3)
- added R11: 100, Resistor_SMD:R_0603_1608Metric, F.Cu at (87.2, 146.8)
- added R12: 100, Resistor_SMD:R_0603_1608Metric, F.Cu at (87.7, 141.7)
- added R13: 1K, Resistor_SMD:R_0603_1608Metric, F.Cu at (87.7, 144.2)
- added R14: 510, Resistor_SMD:R_0603_1608Metric, F.Cu at (124.6, 107.8)
- added R15: *R0, Resistor_SMD:R_0402_1005Metric, F.Cu at (100.7, 118.0)
- added R16: 10K, Resistor_SMD:R_0603_1608Metric, F.Cu at (91.7, 141.7)
- added R17: 10K, Resistor_SMD:R_0603_1608Metric, F.Cu at (102.1, 127.3)
- added R18: 10K, Resistor_SMD:R_0603_1608Metric, F.Cu at (107.0, 125.3)
- added R19: 10K, Resistor_SMD:R_0603_1608Metric, F.Cu at (118.1, 115.1)
- added R20: 10K, Resistor_SMD:R_0603_1608Metric, F.Cu at (95.7, 136.6)
- added R21: 10K, Resistor_SMD:R_0603_1608Metric, F.Cu at (112.9, 117.0)
- added R5: 2K, Resistor_SMD:R_0603_1608Metric, F.Cu at (80.3, 150.8)
- added R6: 20K, Resistor_SMD:R_0603_1608Metric, F.Cu at (118.1, 112.6)
- added R7: 20K, Resistor_SMD:R_0603_1608Metric, F.Cu at (91.7, 139.2)
- added R8: 20K, Resistor_SMD:R_0603_1608Metric, F.Cu at (112.9, 119.5)
- added R9: 20K, Resistor_SMD:R_0603_1608Metric, F.Cu at (98.8, 132.2)
- added U3: MCP73831-2-OT, Package_TO_SOT_SMD:SOT-23-5, F.Cu at (57.8, 149.1)
- added U4: CH340E, Package_SO:MSOP-10_3x3mm_P0.5mm, F.Cu at (114.9, 108.9)
- added U5: LP5907MFX-3.3, Package_TO_SOT_SMD:SOT-23-5, F.Cu at (94.2, 133.2)
- added U6: 24AA02-OT, Package_SO:TSSOP-8_4.4x3mm_P0.65mm, F.Cu at (50.9, 149.2)
- moved C2 76.6 mm to (107.0, 122.8)
- moved U1 71.1 mm to (106.9, 110.6)
- moved C3 70.3 mm to (106.8, 127.8)
- moved R2 67.8 mm to (111.0, 122.8)
- moved SW1 63.4 mm to (83.3, 115.1)
- moved R1 62.3 mm to (102.8, 129.8)
- moved R3 53.9 mm to (95.7, 139.1)
- moved U2 43.3 mm to (47.2, 107.3)
- moved R4 43.2 mm to (83.2, 146.3)
- moved J1 40.9 mm to (96.6, 112.3)
- moved J2 40.0 mm to (85.1, 129.6)
- moved J3 17.9 mm to (55.7, 141.4)
- moved L1 17.5 mm to (62.7, 151.0)
- moved C1 14.7 mm to (76.1, 151.1)
Connections:
- net Net-(J1-PadA4) renamed USB_VCC
- J1 pad A1: Net-(J1-PadA1) -> GND
- J1 pad A12: Net-(J1-PadA1) -> GND
- J1 pad A6: unconnected-(J1-PadA6) -> Net-(J1-PadA6)
- J1 pad A7: unconnected-(J1-PadA7) -> Net-(J1-PadA7)
- J1 pad B1: Net-(J1-PadA1) -> GND
- J1 pad B12: Net-(J1-PadA1) -> GND
- J1 pad B6: unconnected-(J1-PadB6) -> Net-(J1-PadA6)
- J1 pad B7: unconnected-(J1-PadB7) -> Net-(J1-PadA7)
- J2 pad R1: (no net) -> unconnected-(J2-PadR1)
- J2 pad R2: (no net) -> GND
- J3 pad R1: (no net) -> unconnected-(J3-PadR1)
- J3 pad R2: (no net) -> GND
- U1 pad 17: unconnected-(U1-Pad17) -> IIC_SCL
- U1 pad 18: unconnected-(U1-Pad18) -> IIC_SDL
- U2 pad 1: unconnected-(U2-Pad1) -> GND
- U2 pad 2: unconnected-(U2-Pad2) -> VCC
- U2 pad 3: unconnected-(U2-Pad3) -> IIC_SCL
- U2 pad 4: unconnected-(U2-Pad4) -> IIC_SDL

Commit message: UPDATA PCB Signed-off-by: kevin <kevin@lmve.net>
Parts:
- added C12: 10uF, Capacitor_SMD:C_1206_3216Metric, F.Cu at (121.4, 104.1)
- added C13: 10uF, Capacitor_SMD:C_1206_3216Metric, F.Cu at (143.2, 82.6)
- added D6: LED, LED_SMD:LED_0603_1608Metric, F.Cu at (153.0, 79.8)
- added R22: 1K, Resistor_SMD:R_0603_1608Metric, F.Cu at (131.4, 103.0)
- added R23: 1K, Resistor_SMD:R_0603_1608Metric, F.Cu at (150.5, 87.3)
- added R24: 510, Resistor_SMD:R_0603_1608Metric, F.Cu at (129.5, 108.1)
- J2: value AudioJack3_Ground -> INPUT
- J3: value AudioJack3_Ground -> OUTPUT
- moved U3 124.5 mm to (156.1, 72.7)
- moved C11 119.3 mm to (160.9, 72.0)
- moved R12 104.4 mm to (165.1, 71.8)
- moved R13 100.8 mm to (160.6, 74.8)
- moved C4 98.6 mm to (155.7, 76.5)
- moved C7 94.3 mm to (148.3, 84.5)
- moved Q2 94.3 mm to (148.5, 80.8)
- moved L1 85.5 mm to (131.7, 100.4)
- moved R7 83.6 mm to (152.9, 82.4)
- moved R5 83.0 mm to (140.8, 94.0)
- moved D1 76.6 mm to (139.7, 99.0)
- moved C6 76.0 mm to (136.7, 87.4)
- moved C9 75.1 mm to (126.5, 105.0)
- moved R1 72.4 mm to (157.0, 81.7)
- moved R15 61.2 mm to (152.0, 84.6)
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Connections:
- net BAT renamed Net-(C8-Pad1)
- J2 pad R1: unconnected-(J2-PadR1) -> TICK_A
- J2 pad T: unconnected-(J2-PadT) -> TICK_B
- J3 pad R1: unconnected-(J3-PadR1) -> Net-(C12-Pad1)
- J3 pad T: unconnected-(J3-PadT) -> Net-(C13-Pad1)
- SW1 pad S1: SW1 -> K1
- U1 pad 10: unconnected-(U1-Pad10) -> PWM
- U1 pad 11: unconnected-(U1-Pad11) -> MUTE
- U1 pad 14: SW1 -> K1_DET
- U1 pad 19: unconnected-(U1-Pad19) -> PWR_EN
- U1 pad 2: unconnected-(U1-Pad2) -> TICK_A
- U1 pad 20: unconnected-(U1-Pad20) -> RUN_LED
- U1 pad 3: unconnected-(U1-Pad3) -> TICK_B
- U1 pad 6: unconnected-(U1-Pad6) -> BAT_ADC
- U1 pad 7: unconnected-(U1-Pad7) -> BAT_CHG_DET
- U1 pad 8: unconnected-(U1-Pad8) -> RXD
- U1 pad 9: unconnected-(U1-Pad9) -> TXD

Commit message: UPDATA PCB Signed-off-by: kevin <kevin@lmve.net>
Parts:
- added J4: Conn_01x02_Female, MY:SIP-2, F.Cu at (128.0, 156.1)
- J2: moved to B.Cu
- U6: footprint Package_SO:TSSOP-8_4.4x3mm_P0.65mm -> Package_TO_SOT_SMD:SOT-23-5
- moved U3 96.0 mm to (110.9, 157.4)
- moved R10 95.0 mm to (111.5, 152.7), turned to 180 degrees
- moved R12 93.1 mm to (116.1, 150.9)
- moved C4 90.4 mm to (108.8, 153.7), turned to -90 degrees
- moved Q2 89.0 mm to (106.2, 159.1), turned to 90 degrees
- moved R13 85.1 mm to (115.2, 146.7), turned to -90 degrees
- moved C7 82.7 mm to (114.1, 159.8), turned to 90 degrees
- moved C6 77.5 mm to (110.7, 160.4), turned to 180 degrees
- moved U4 71.5 mm to (111.0, 150.0), turned to 180 degrees
- moved R14 68.3 mm to (109.7, 147.3)
- moved R5 67.1 mm to (111.5, 154.4)
- moved D2 58.7 mm to (128.0, 148.6), turned to 180 degrees
- moved C5 54.9 mm to (114.3, 155.2), turned to -90 degrees
- moved D3 42.6 mm to (128.0, 150.3)
- moved R11 34.6 mm to (116.1, 149.3)
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Connections:
- J1 pad S1: unconnected-(J1-PadS1) -> GND
Routing:
- net GND: track 0.00 -> 48.1 mm
- net USB_VCC: track 0.00 -> 26.0 mm
- net BAT_IN: track 0.00 -> 24.5 mm
- net Net-(D2-Pad2): track 0.00 -> 22.4 mm
- net Net-(J1-PadA6): track 0.00 -> 8.00 mm
- net VCC: track 0.00 -> 7.90 mm
- net Net-(J1-PadA7): track 0.00 -> 7.88 mm
- net Net-(R12-Pad1): track 0.00 -> 5.55 mm
- net Net-(R11-Pad1): track 0.00 -> 5.38 mm
- net BAT_CHG_DET: track 0.00 -> 4.13 mm
- net Net-(R5-Pad2): track 0.00 -> 2.17 mm
- net Net-(C4-Pad1): track 0.00 -> 1.75 mm
- net Net-(R14-Pad1): track 0.00 -> 1.73 mm
- net (no net): vias 0 -> 4

Commit message: 又是12点了，下班后累的不想动，随便折腾一会又该睡觉了 明天摸鱼画吧
画好了电源部分。。
Signed-off-by: kevin <kevin@lmve.net>
Parts:
- moved C11 96.2 mm to (106.8, 151.5), turned to -90 degrees
- moved R7 91.4 mm to (103.5, 159.3), turned to -90 degrees
- moved R6 87.0 mm to (98.1, 159.7), turned to -90 degrees
- moved D5 78.4 mm to (96.6, 156.8), turned to 90 degrees
- moved D1 74.6 mm to (96.6, 159.9), turned to 90 degrees
- moved Q1 73.9 mm to (100.8, 159.4)
- moved C8 72.2 mm to (103.3, 154.8), turned to 180 degrees
- moved U5 56.4 mm to (101.3, 151.5)
- moved D4 55.8 mm to (98.1, 156.8), turned to -90 degrees
- moved C3 55.4 mm to (107.3, 145.6), turned to 180 degrees
- moved R3 54.4 mm to (104.2, 147.7), turned to 180 degrees
- moved C9 53.9 mm to (106.7, 155.1), turned to 90 degrees
- moved R9 51.4 mm to (100.1, 155.1), turned to 90 degrees
- moved R8 49.4 mm to (102.8, 156.9), turned to 180 degrees
- moved C10 38.6 mm to (104.6, 150.9), turned to -90 degrees
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Routing:
- net GND: track 48.1 -> 97.3 mm
- net Net-(C3-Pad1): track 0.00 -> 21.6 mm
- net Net-(C2-Pad1): track 0.00 -> 21.0 mm
- net Net-(D3-Pad1): track 0.00 -> 17.4 mm, vias 0 -> 2
- net Net-(C8-Pad1): track 0.00 -> 16.4 mm
- net VCC: track 7.90 -> 19.6 mm
- net Net-(D4-Pad2): track 0.00 -> 9.19 mm
- net Net-(D1-Pad1): track 0.00 -> 4.34 mm
- net BAT_IN: track 24.5 -> 28.5 mm
- net BAT_ADC: track 0.00 -> 2.44 mm
- net K1: track 0.00 -> 2.09 mm
- net USB_VCC: track 26.0 -> 24.1 mm
- net Net-(D2-Pad2): track 22.4 -> 20.5 mm
